File: Hardware/Sensor_Board/LCD.kicad_sch (KiCad schematic)
At the start: 1 part, among them U4 LCD

Commit message: Add files via upload
Connections:
- net GND: now also U4.2 (VDD)
- net 5V: now reaches U4.1 (VCC)
Changed lines of the file:
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@@
 	(generator_version "9.0")
 	(paper "A4")
+	(wire
+		(pts
+			(xy 31.75 85.09) (xy 63.5 85.09)
+		)
+		(stroke
+			(width 0)
+			(type default)
+		)
+	)
+	(wire
+		(pts
+			(xy 76.2 87.63) (xy 76.2 66.04)
+		)
+		(stroke
+			(width 0)
+			(type default)
+		)
+	)
+	(wire
+		(pts
+			(xy 31.75 87.63) (xy 76.2 87.63)
+		)
+		(stroke
+			(width 0)
+			(type default)
+		)
+	)
+	(wire
+		(pts
+			(xy 63.5 85.09) (xy 63.5 63.5)
+		)
+		(stroke
+			(width 0)
+			(type default)
+		)
+	)
 	(hierarchical_label "GND"
 		(shape input)
-		(at 31.75 80.01 180)
+		(at 31.75 85.09 180)
 		(effects
 			(font
@@
 		)
 	)
-	(hierarchical_label "3.3V"
+	(hierarchical_label "5V"
 		(shape input)
-		(at 31.75 17.78 180)
+		(at 31.75 87.63 180)
 		(effects
 			(font
@@
 	(symbol
 		(lib_id "Symbols:LCD240X320")
-		(at 90.17 97.79 0)
+		(at 91.44 90.17 0)
 		(unit 1)
 		(exclude_from_sim no)
@@
 		(fields_autoplaced yes)
 		(property "Reference" "U4"
-			(at 66.04 37.084 0)
+			(at 67.31 29.464 0)
 			(effects
 				(font
@@
 		)
 		(property "Value" "LCD"
-			(at 81.28 55.8799 0)
+			(at 82.55 48.2599 0)
 			(effects
 				(font
@@
 		)
 		(property "Footprint" "Display:LCD-016N002L"
-			(at 72.898 79.248 0)
+			(at 74.168 71.628 0)
 			(effects
 				(font
@@
 		)
 		(property "Datasheet" "http://www.vishay.com/docs/37299/37299.pdf"
-			(at 60.198 116.586 0)
+			(at 61.468 108.966 0)
 			(do_not_autoplace yes)
 			(effects
@@
 		)
 		(property "Description" "LCD 12x2, 8 bit parallel bus, 3V or 5V VDD"
-			(at 61.214 114.808 0)
+			(at 62.484 107.188 0)
 			(do_not_autoplace yes)
 			(effects
