File: Schematics/Hardware/LED_Board/CPE495-LED-Driver-Board.kicad_sch (KiCad schematic)
At the start: 7 parts, among them J1 Conn_02x20_Odd_Even, J2 Conn_02x08_Odd_Even, J3 Conn_02x13_Odd_Even, U1 74AHCT245, U2 74AHCT245

Commit message: Add files via upload
Parts:
- removed J1: Conn_02x20_Odd_Even, Connector_IDC:IDC-Header_2x20_P2.54mm_Vertical, symbol Connector_Generic:Conn_02x20_Odd_Even
- removed J3: Conn_02x13_Odd_Even, Connector_PinHeader_2.54mm:PinHeader_2x13_P2.54mm_Vertical, symbol Connector_Generic:Conn_02x13_Odd_Even
- added Alinx-J2, Terasic-J1: Conn_02x20_Odd_Even, Connector_IDC:IDC-Header_2x20_P2.54mm_Vertical, symbol Connector_Generic:Conn_02x20_Odd_Even
- added H1, H2, H3, H4: MountingHole_Pad, MountingHole:MountingHole_2.5mm_Pad_Via, symbol Mechanical:MountingHole_Pad
Connections:
- net +3.3V: now also Alinx-J2.39 (Pin_39), Alinx-J2.40 (Pin_40), Terasic-J1.29 (Pin_29)
- net +5V: now also Alinx-J2.2 (Pin_2), Terasic-J1.11 (Pin_11)
- net A: now also U1.13 (B5); no longer U1.11 (B7)
- net B: now also U1.11 (B7); no longer U2.18 (B0)
- net B1: now also U2.15 (B3); no longer U1.16 (B2)
- net B2: now also U2.18 (B0); no longer U1.13 (B5)
- net C: now also U1.15 (B3); no longer U2.17 (B1)
- net CLK: now also U1.17 (B1); no longer U2.15 (B3)
- net D: now also U1.14 (B4); no longer U2.16 (B2)
- net G1: now also U2.13 (B5); no longer U1.17 (B1)
- net G2: now also U2.16 (B2); no longer U1.14 (B4)
- net GND: now also Alinx-J2.1 (Pin_1), Alinx-J2.37 (Pin_37), Alinx-J2.38 (Pin_38), H1.1, H2.1, H3.1, H4.1, Terasic-J1.12 (Pin_12), Terasic-J1.30 (Pin_30)
- net LATCH: now also U1.16 (B2); no longer U2.14 (B4)
- net OE: now also U1.18 (B0); no longer U2.13 (B5)
- net R1: now also U2.14 (B4); no longer U1.18 (B0)
- net R2: now also U2.17 (B1); no longer U1.15 (B3)
- net GPIO0 (AB22) (V10) renamed GPIO33 (AH26) (Y3) (17P)
- net GPIO33 (AH26) (Y3) (17P): now also Alinx-J2.36 (Pin_36), Terasic-J1.38 (Pin_38)
- net GPIO1 (AC15) (W10) renamed GPIO32 (AF20) (AB3) (17N)
- net GPIO32 (AF20) (AB3) (17N): now also Alinx-J2.35 (Pin_35), Terasic-J1.37 (Pin_37)
- net GPIO2 (AB21) (V9) renamed GPIO31 (AG23) (Y4) (16P)
- net GPIO31 (AG23) (Y4) (16P): now also Alinx-J2.34 (Pin_34), Terasic-J1.36 (Pin_36)
- net GPIO29 (AF26) (Y5) renamed GPIO6 (AD21) (V7) (4N)
- net GPIO6 (AD21) (V7) (4N): now also Alinx-J2.9 (Pin_9), Terasic-J1.7 (Pin_7)
- net GPIO3 (Y17) (W9) renamed GPIO30 (AE20) (AA5) (16N)
- net GPIO30 (AE20) (AA5) (16N): now also Alinx-J2.33 (Pin_33), Terasic-J1.35 (Pin_35)
- net GPIO30 (AE20) (AA5) renamed GPIO5 (Y16) (W8) (3P)
- net GPIO5 (Y16) (W8) (3P): now also Alinx-J2.8 (Pin_8), Terasic-J1.6 (Pin_6)
- net GPIO31 (AG23) (Y4) renamed GPIO4 (AC21) (V8) (3N)
- net GPIO4 (AC21) (V8) (3N): now also Alinx-J2.7 (Pin_7), Terasic-J1.5 (Pin_5)
- net GPIO32 (AF20) (AB3) renamed GPIO3 (Y17) (W9) (2P)
- net GPIO3 (Y17) (W9) (2P): now also Alinx-J2.6 (Pin_6), Terasic-J1.4 (Pin_4)
- net GPIO33 (AH26) (Y3) renamed GPIO2 (AB21) (V9) (2N)
- net GPIO2 (AB21) (V9) (2N): now also Alinx-J2.5 (Pin_5), Terasic-J1.3 (Pin_3)
- net GPIO34 (AH23) (AB2) renamed GPIO1 (AC15) (W10) (1P)
- net GPIO1 (AC15) (W10) (1P): now also Alinx-J2.4 (Pin_4), Terasic-J1.2 (Pin_2)
- net GPIO35 (AG26) (AA2) renamed GPIO0 (AB22) (V10) (1N)
- net GPIO0 (AB22) (V10) (1N): now also Alinx-J2.3 (Pin_3), Terasic-J1.1 (Pin_1)
- net GPIO4 (AC21) (V8) renamed GPIO29 (AF26) (Y5) (15P)
- net GPIO29 (AF26) (Y5) (15P): now also Alinx-J2.32 (Pin_32), Terasic-J1.34 (Pin_34)
- net GPIO5 (Y16) (W8) renamed GPIO28 (AH22) (AA6) (15N)
- net GPIO28 (AH22) (AA6) (15N): now also Alinx-J2.31 (Pin_31), Terasic-J1.33 (Pin_33)
- new net GPIO10 (AC19) (W5) (6N): Alinx-J2.13 (Pin_13), Terasic-J1.13 (Pin_13)
- new net GPIO11 (AF16) (AA15) (6P): Alinx-J2.14 (Pin_14), Terasic-J1.14 (Pin_14)
- new net GPIO12 (AD19) (AA14) (7N): Alinx-J2.15 (Pin_15), Terasic-J1.15 (Pin_15)
- new net GPIO13 (AF15) (W13) (7P): Alinx-J2.16 (Pin_16), Terasic-J1.16 (Pin_16)
- new net GPIO14 (AF24) (W12) (8N): Alinx-J2.17 (Pin_17), Terasic-J1.17 (Pin_17)
- new net GPIO15 (AE21) (AB13) (8P): Alinx-J2.18 (Pin_18), Terasic-J1.18 (Pin_18)
- new net GPIO16 (AF25) (AB12) (9N): Alinx-J2.19 (Pin_19), Terasic-J1.19 (Pin_19)
- new net GPIO17 (AC22) (Y11) (9P): Alinx-J2.20 (Pin_20), Terasic-J1.20 (Pin_20)
- new net GPIO18 (AE22) (AB11) (10N): Alinx-J2.21 (Pin_21), Terasic-J1.21 (Pin_21)
- new net GPIO19 (AF21) (W11) (10P): Alinx-J2.22 (Pin_22), Terasic-J1.22 (Pin_22)
- new net GPIO20 (AF22) (AB10) (11N): Alinx-J2.23 (Pin_23), Terasic-J1.23 (Pin_23)
- new net GPIO21 (AD22) (AA10) (11P): Alinx-J2.24 (Pin_24), Terasic-J1.24 (Pin_24)
- new net GPIO22 (AG25) (AA9) (12N): Alinx-J2.25 (Pin_25), Terasic-J1.25 (Pin_25)
- new net GPIO23 (AD25) (Y8) (12P): Alinx-J2.26 (Pin_26), Terasic-J1.26 (Pin_26)
- new net GPIO24 (AH25) (AA8) (13N): Alinx-J2.27 (Pin_27), Terasic-J1.27 (Pin_27)
- new net GPIO25 (AE25) (Y7) (13P): Alinx-J2.28 (Pin_28), Terasic-J1.28 (Pin_28)
- new net GPIO26 (AG22) (AA7) (14N): Alinx-J2.29 (Pin_29), Terasic-J1.31 (Pin_31)
- new net GPIO27 (AE24) (Y6) (14P): Alinx-J2.30 (Pin_30), Terasic-J1.32 (Pin_32)
- new net GPIO34 (AH23) (AB2) (NC): Terasic-J1.39 (Pin_39)
- new net GPIO35 (AG26) (AA2) (NC): Terasic-J1.40 (Pin_40)
- new net GPIO7 (AE16) (W7) (4P): Alinx-J2.10 (Pin_10), Terasic-J1.8 (Pin_8)
- new net GPIO8 (AD15) (W6) (5N): Alinx-J2.11 (Pin_11), Terasic-J1.9 (Pin_9)
- new net GPIO9 (AE15) (V5) (5P): Alinx-J2.12 (Pin_12), Terasic-J1.10 (Pin_10)
- no-connect marks 0 -> 3
