File: Schematics/Hardware/LED_Board/CPE495-LED-Driver-Board.kicad_pcb (KiCad board)
At the start: 2 copper layers, 58.4 x 66 mm, 7 parts, among them J1 Conn_02x20_Odd_Even, J2 Conn_02x08_Odd_Even, J3 Conn_02x13_Odd_Even, U1 74AHCT245, U2 74AHCT245

Commit message: Add files via upload
Parts:
- removed J1: Conn_02x20_Odd_Even, Connector_IDC:IDC-Header_2x20_P2.54mm_Vertical
- removed J3: Conn_02x13_Odd_Even, Connector_PinHeader_2.54mm:PinHeader_2x13_P2.54mm_Vertical
- added Alinx-J2: Conn_02x20_Odd_Even, Connector_IDC:IDC-Header_2x20_P2.54mm_Vertical, F.Cu at (156.3, 77.2)
- added H1: MountingHole_Pad, MountingHole:MountingHole_2.5mm_Pad_Via, F.Cu at (201.2, 66.1)
- added H2: MountingHole_Pad, MountingHole:MountingHole_2.5mm_Pad_Via, F.Cu at (142.5, 66.5)
- added H3: MountingHole_Pad, MountingHole:MountingHole_2.5mm_Pad_Via, F.Cu at (201.0, 135.1)
- added H4: MountingHole_Pad, MountingHole:MountingHole_2.5mm_Pad_Via, F.Cu at (142.5, 135.1)
- added Terasic-J1: Conn_02x20_Odd_Even, Connector_IDC:IDC-Header_2x20_P2.54mm_Vertical, F.Cu at (142.9, 77.2)
- moved J2 19.4 mm to (200.0, 112.9), turned to 180 degrees
Connections:
- U1 pad 11: A -> B
- U1 pad 13: B2 -> A
- U1 pad 14: G2 -> D
- U1 pad 15: R2 -> C
- U1 pad 16: B1 -> LATCH
- U1 pad 17: G1 -> CLK
- U1 pad 18: R1 -> OE
- U1 pad 2: GPIO35 (AG26) (AA2) -> GPIO0 (AB22) (V10) (1N)
- U1 pad 3: GPIO34 (AH23) (AB2) -> GPIO1 (AC15) (W10) (1P)
- U1 pad 4: GPIO33 (AH26) (Y3) -> GPIO2 (AB21) (V9) (2N)
- U1 pad 5: GPIO32 (AF20) (AB3) -> GPIO3 (Y17) (W9) (2P)
- U1 pad 6: GPIO31 (AG23) (Y4) -> GPIO4 (AC21) (V8) (3N)
- U1 pad 7: GPIO30 (AE20) (AA5) -> GPIO5 (Y16) (W8) (3P)
- U1 pad 9: GPIO29 (AF26) (Y5) -> GPIO6 (AD21) (V7) (4N)
- U2 pad 13: OE -> G1
- U2 pad 14: LATCH -> R1
- U2 pad 15: CLK -> B1
- U2 pad 16: D -> G2
- U2 pad 17: C -> R2
- U2 pad 18: B -> B2
- U2 pad 2: GPIO5 (Y16) (W8) -> GPIO28 (AH22) (AA6) (15N)
- U2 pad 3: GPIO4 (AC21) (V8) -> GPIO29 (AF26) (Y5) (15P)
- U2 pad 4: GPIO3 (Y17) (W9) -> GPIO30 (AE20) (AA5) (16N)
- U2 pad 5: GPIO2 (AB21) (V9) -> GPIO31 (AG23) (Y4) (16P)
- U2 pad 6: GPIO1 (AC15) (W10) -> GPIO32 (AF20) (AB3) (17N)
- U2 pad 7: GPIO0 (AB22) (V10) -> GPIO33 (AH26) (Y3) (17P)
Routing:
- net +3.3V: track 90.8 -> 30.8 mm
- net GPIO28 (AH22) (AA6): track 59.8 -> 0.00 mm
- net GPIO27 (AE24) (Y6): track 58.2 -> 0.00 mm
- net GPIO26 (AG22) (AA7): track 56.2 -> 0.00 mm
- net GPIO25 (AE25) (Y7): track 52.1 -> 0.00 mm
- net GPIO24 (AH25) (AA8): track 50.1 -> 0.00 mm
- net GPIO23 (AD25) (Y8): track 48.5 -> 0.00 mm
- net GPIO22 (AG25) (AA9): track 46.5 -> 0.00 mm
- net GPIO21 (AD22) (AA10): track 44.9 -> 0.00 mm
- net GPIO0 (AB22) (V10) (1N): track 0.00 -> 43.5 mm
- net GPIO2 (AB21) (V9) (2N): track 0.00 -> 42.9 mm
- net GPIO20 (AF22) (AB10): track 42.9 -> 0.00 mm
- net GPIO4 (AC21) (V8) (3N): track 0.00 -> 42.4 mm
- net GPIO6 (AD21) (V7) (4N): track 0.00 -> 42.2 mm
- net GPIO19 (AF21) (W11): track 41.4 -> 0.00 mm
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Other:
- board size 58.4 x 66 mm -> 69.2 x 79.9 mm
- board text added: "LED Driver Board v0.5"
- board text removed: "LED Driver Board v0.3"
- board text removed: "WayWayWay"

Commit message: Add files via upload
Parts:
- added G***: LOGO, LOGO, F.Cu at (175.5, 136.5)
- added G***: LOGO, LOGO, B.Cu at (187.5, 133.0)
Other:
- board text added: "A.L.D.L."
- board text added: "https://github.com/dmc0022/ALDL_repo"
